File: SAP-BE/ALU.sch (KiCad schematic (older format))
At the start: 5 parts, among them U1 74LS86, U2 74LS86, U3 74LS283, U4 74LS283, U5 74LS245

Commit message: Update with conditional flags
Parts:
- added U46: 7402, symbol 7402
- added U47: 74LS08, symbol 74LS08
Connections:
- net labels added: ZERO, sum0, sum1, sum2, sum3, sum4, sum5, sum6, sum7
- wire segments 92 -> 120
Other:
- note added: "Zero compute"
- moved on the sheet: U1A, U1B, U1C, U1D, U2A, U2B, U2C, U2D, U3, U4, U5
