File: SAP-BE/instructionregister.sch (KiCad schematic (older format))
At the start: 11 parts, among them U15 74LS173, U16 74LS173, U17 74LS245

Commit message: Update with changes for reset
Connections:
- net labels added: RESET
Changed lines of the file:
@@
 	3700 2050 3800 2150
 $Comp
-L VCC #PWR67
+L VCC #PWR069
 U 1 1 590A466E
 P 6450 3750
-F 0 "#PWR67" H 6450 3600 50  0001 C CNN
+F 0 "#PWR069" H 6450 3600 50  0001 C CNN
 F 1 "VCC" H 6450 3900 50  0000 C CNN
 F 2 "" H 6450 3750 50  0000 C CNN
@@
 Text HLabel 2750 2650 0    60   Input ~ 0
 ~RENABLE
-Text HLabel 2750 2350 0    60   Input ~ 0
-CLR
 Text HLabel 2750 2050 0    60   Input ~ 0
 ~LOAD
@@
 ~LOAD
 $Comp
-L GND #PWR68
+L GND #PWR070
 U 1 1 590D3ED6
 P 8650 5250
-F 0 "#PWR68" H 8650 5000 50  0001 C CNN
+F 0 "#PWR070" H 8650 5000 50  0001 C CNN
 F 1 "GND" H 8650 5100 50  0000 C CNN
 F 2 "" H 8650 5250 50  0000 C CNN
@@
 r[0..7]
 $Comp
-L GND #PWR66
+L GND #PWR071
 U 1 1 59133E3E
 P 6250 3550
-F 0 "#PWR66" H 6250 3300 50  0001 C CNN
+F 0 "#PWR071" H 6250 3300 50  0001 C CNN
 F 1 "GND" H 6250 3400 50  0000 C CNN
 F 2 "" H 6250 3550 50  0000 C CNN
@@
 Wire Wire Line
 	6250 3550 6550 3550
+Text HLabel 2750 2350 0    60   Input ~ 0
+RESET
 $EndSCHEMATC
