File: SAP-BE/status.sch (KiCad schematic (older format))
At the start: 32 parts, among them U28 74HC04, U29 74HC04

Commit message: Update with conditional flags
Parts:
- added D67: LED, LEDs:LED-5MM, symbol LED
- added R30: 470, Resistors_THT:Resistor_Horizontal_RM7mm, symbol R
Connections:
- net GND: now also R30.2
- net FI: now reaches U29.3
- net FI: now also D67.2 (A)
- net ~FI: now reaches U29.4
- new net: D67.1 (K), R30.1
- no-connect marks 4 -> 2
Other:
- moved on the sheet: U29B
Changed lines of the file:
@@
 $Descr A4 11693 8268
 encoding utf-8
-Sheet 11 11
+Sheet 11 12
 Title "Simple As Possible computer by Ben Eater"
 Date "2017-05-10"
@@
 L 74HC04 U29
 U 2 1 591355A0
-P 8600 5100
-F 0 "U29" H 8750 5200 50  0000 C CNN
-F 1 "74HC04" H 8800 5000 50  0000 C CNN
-F 2 "Housings_DIP:DIP-14_W7.62mm_LongPads" H 8600 5100 50  0001 C CNN
-F 3 "" H 8600 5100 50  0000 C CNN
-	2    8600 5100
+P 6850 4600
+F 0 "U29" H 7000 4700 50  0000 C CNN
+F 1 "74HC04" H 7050 4500 50  0000 C CNN
+F 2 "Housings_DIP:DIP-14_W7.62mm_LongPads" H 6850 4600 50  0001 C CNN
+F 3 "" H 6850 4600 50  0000 C CNN
+	2    6850 4600
 	1    0    0    -1
 $EndComp
@@
 	2300 1000 2500 1000
 $Comp
-L GND #PWR072
+L GND #PWR074
 U 1 1 59135B35
 P 2450 1750
-F 0 "#PWR072" H 2450 1500 50  0001 C CNN
+F 0 "#PWR074" H 2450 1500 50  0001 C CNN
 F 1 "GND" H 2450 1600 50  0000 C CNN
 F 2 "" H 2450 1750 50  0000 C CNN
@@
 $EndComp
 $Comp
-L GND #PWR073
+L GND #PWR075
 U 1 1 59136020
 P 6350 3550
-F 0 "#PWR073" H 6350 3300 50  0001 C CNN
+F 0 "#PWR075" H 6350 3300 50  0001 C CNN
 F 1 "GND" H 6350 3400 50  0000 C CNN
 F 2 "" H 6350 3550 50  0000 C CNN
@@
 $EndComp
 $Comp
-L GND #PWR074
+L GND #PWR076
 U 1 1 591365E5
 P 4650 1750
-F 0 "#PWR074" H 4650 1500 50  0001 C CNN
+F 0 "#PWR076" H 4650 1500 50  0001 C CNN
 F 1 "GND" H 4650 1600 50  0000 C CNN
 F 2 "" H 4650 1750 50  0000 C CNN
@@
 	6200 1000 6400 1000
 $Comp
-L GND #PWR075
+L GND #PWR077
 U 1 1 59136DC1
 P 6350 1750
-F 0 "#PWR075" H 6350 1500 50  0001 C CNN
+F 0 "#PWR077" H 6350 1500 50  0001 C CNN
 F 1 "GND" H 6350 1600 50  0000 C CNN
 F 2 "" H 6350 1750 50  0000 C CNN
@@
 	8200 1000 8400 1000
 $Comp
-L GND #PWR076
+L GND #PWR078
 U 1 1 59139E9F
 P 8350 1750
-F 0 "#PWR076" H 8350 1500 50  0001 C CNN
+F 0 "#PWR078" H 8350 1500 50  0001 C CNN
 F 1 "GND" H 8350 1600 50  0000 C CNN
 F 2 "" H 8350 1750 50  0000 C CNN
@@
 	9850 1000 10050 1000
 $Comp
-L GND #PWR077
+L GND #PWR079
 U 1 1 5913AABA
 P 10000 1750
-F 0 "#PWR077" H 10000 1500 50  0001 C CNN
+F 0 "#PWR079" H 10000 1500 50  0001 C CNN
 F 1 "GND" H 10000 1600 50  0000 C CNN
 F 2 "" H 10000 1750 50  0000 C CNN
@@
 	750  2800 950  2800
 $Comp
-L GND #PWR078
+L GND #PWR080
 U 1 1 5913AE3F
 P 900 3550
-F 0 "#PWR078" H 900 3300 50  0001 C CNN
+F 0 "#PWR080" H 900 3300 50  0001 C CNN
 F 1 "GND" H 900 3400 50  0000 C CNN
 F 2 "" H 900 3550 50  0000 C CNN
@@
 	2300 2800 2500 2800
 $Comp
-L GND #PWR079
+L GND #PWR081
 U 1 1 5913C2F6
 P 2450 3550
-F 0 "#PWR079" H 2450 3300 50  0001 C CNN
+F 0 "#PWR081" H 2450 3300 50  0001 C CNN
 F 1 "GND" H 2450 3400 50  0000 C CNN
 F 2 "" H 2450 3550 50  0000 C CNN
@@
 	4500 2800 4700 2800
 $Comp
-L GND #PWR080
+L GND #PWR082
 U 1 1 591416A1
 P 4650 3550
-F 0 "#PWR080" H 4650 3300 50  0001 C CNN
+F 0 "#PWR082" H 4650 3300 50  0001 C CNN
 F 1 "GND" H 4650 3400 50  0000 C CNN
 F 2 "" H 4650 3550 50  0000 C CNN
@@
 $EndComp
 $Comp
-L GND #PWR081
+L GND #PWR083
 U 1 1 59141903
 P 8400 3550
-F 0 "#PWR081" H 8400 3300 50  0001 C CNN
+F 0 "#PWR083" H 8400 3300 50  0001 C CNN
 F 1 "GND" H 8400 3400 50  0000 C CNN
 F 2 "" H 8400 3550 50  0000 C CNN
@@
 $EndComp
 $Comp
-L GND #PWR082
+L GND #PWR084
 U 1 1 5914A0BC
 P 10000 3550
-F 0 "#PWR082" H 10000 3300 50  0001 C CNN
+F 0 "#PWR084" H 10000 3300 50  0001 C CNN
 F 1 "GND" H 10000 3400 50  0000 C CNN
 F 2 "" H 10000 3550 50  0000 C CNN
@@
 $EndComp
 $Comp
-L GND #PWR083
+L GND #PWR085
 U 1 1 59150B97
 P 900 5350
-F 0 "#PWR083" H 900 5100 50  0001 C CNN
+F 0 "#PWR085" H 900 5100 50  0001 C CNN
 F 1 "GND" H 900 5200 50  0000 C CNN
 F 2 "" H 900 5350 50  0000 C CNN
@@
 $EndComp
 $Comp
-L GND #PWR084
+L GND #PWR086
 U 1 1 591547E6
 P 2450 5350
-F 0 "#PWR084" H 2450 5100 50  0001 C CNN
+F 0 "#PWR086" H 2450 5100 50  0001 C CNN
 F 1 "GND" H 2450 5200 50  0000 C CNN
 F 2 "" H 2450 5350 50  0000 C CNN
@@
 $EndComp
 $Comp
-L GND #PWR085
+L GND #PWR087
 U 1 1 5915490F
 P 4650 5350
-F 0 "#PWR085" H 4650 5100 50  0001 C CNN
+F 0 "#PWR087" H 4650 5100 50  0001 C CNN
 F 1 "GND" H 4650 5200 50  0000 C CNN
 F 2 "" H 4650 5350 50  0000 C CNN
@@
 $EndComp
 $Comp
-L GND #PWR086
+L GND #PWR088
 U 1 1 5915A814
 P 900 1750
-F 0 "#PWR086" H 900 1500 50  0001 C CNN
+F 0 "#PWR088" H 900 1500 50  0001 C CNN
 F 1 "GND" H 900 1600 50  0000 C CNN
 F 2 "" H 900 1750 50  0000 C CNN
@@
 NoConn ~ 10600 5050
 NoConn ~ 9700 5050
-NoConn ~ 9050 5100
-NoConn ~ 8150 5100
+Text HLabel 6150 4600 0    60   Input ~ 0
+FI
+Text HLabel 7350 4600 2    60   Output ~ 0
+~FI
+Wire Wire Line
+	7350 4600 7300 4600
+Wire Wire Line
+	6400 4600 6150 4600
+$Comp
+L LED D67
+U 1 1 5AD0ADC1
+P 6350 4800
+F 0 "D67" H 6350 4900 50  0000 C CNN
+F 1 "LED" H 6350 4700 50  0000 C CNN
+F 2 "LEDs:LED-5MM" H 6350 4800 50  0001 C CNN
+F 3 "" H 6350 4800 50  0000 C CNN
+	1    6350 4800
+	0    -1   -1   0
+$EndComp
+$Comp
+L R R30
+U 1 1 5AD0ADCC
+P 6350 5150
+F 0 "R30" V 6430 5150 50  0000 C CNN
+F 1 "470" V 6350 5150 50  0000 C CNN
+F 2 "Resistors_THT:Resistor_Horizontal_RM7mm" V 6280 5150 50  0001 C CNN
+F 3 "" H 6350 5150 50  0000 C CNN
+	1    6350 5150
+	1    0    0    -1
+$EndComp
+$Comp
+L GND #PWR089
+U 1 1 5AD0ADD7
+P 6350 5350
+F 0 "#PWR089" H 6350 5100 50  0001 C CNN
+F 1 "GND" H 6350 5200 50  0000 C CNN
+F 2 "" H 6350 5350 50  0000 C CNN
+F 3 "" H 6350 5350 50  0000 C CNN
+	1    6350 5350
+	1    0    0    -1
+$EndComp
+Wire Wire Line
+	6350 4650 6350 4600
+Connection ~ 6350 4600
+Wire Wire Line
+	6350 4950 6350 5000
+Wire Wire Line
+	6350 5300 6350 5350
 $EndSCHEMATC
